File: TR4_PGA257(v4.0)/ROHM_PCB_thuc/TR4.brd (EAGLE design)
At the start: 204 x 172 mm, 124 parts, among them IC1 SN74AVC4T774PWR, IC3 SN74AVC4T774PWR, IC4 SN74AVC4T774PWR, IC7 LM1117MP-1.8_NOPB, IC8 LM1117MP-1.8_NOPB, IC9 LM1117MP-1.8_NOPB, J4 2985-6004, J5 2985-6004, Q10 BSH103,235, Q11 BSH103,235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

Commit message: Add files via upload
Parts:
- added R1, R3, R5: 15k, SparkFun-Resistors:0603
- added R2, R4, R6: 6.8k, SparkFun-Resistors:0603
- C14, C16, C18: value 10uF -> 100uF
- IC7, IC8, IC9: value LM1117MP-1.8_NOPB -> LM1117IMPX-ADJ/NOPB
- renumbered JP11 to FLASH, JP12 to USB-UART, JP9 to SD_CARD
Connections:
- net GND: now also R1.1, R2.1, R2.2, R3.1, R4.1, R4.2, R5.1, R6.1, R6.2
- net VDD_1.8_1: now also R1.2
- net VDD_1.8_2: now also R3.2
- net VDD_1.8_3: now also R5.2
Routing:
- net GND: track 1224.2 -> 1239.0 mm
- net VDD_1.8_2: track 22.6 -> 31.2 mm
- net VDD_1.8_3: track 24.4 -> 33.0 mm
- net VDD_1.8_1: track 24.9 -> 33.3 mm
- net VDD_3V3: track 685.2 -> 687.8 mm
Other:
- board text added: "1.8V CHIP"
- board text added: "1.8V CHIP IO"
- board text added: "SD card"
- board text removed: "1.8V CORE"
- board text removed: "1.8V IO CORE"
- board text removed: "FLASH_WP FLASH_SCK FLASH_MOSI FLASH_MISO FLASH_CS FLASH_RESET FLASH_HOLD"
- board text removed: "RX"
- board text removed: "SMA"
- board text removed: "SPI"
- board text removed: "TX"
- board text removed: "UART_RXD"
- board text removed: "UART_TXD"
- board text removed: "USB Power (5V)"
