File: TR4_PGA257(v4.0)/ROHM_PCB_thuc/TR4.sch (EAGLE design)
At the start: 124 parts, among them IC1 SN74AVC4T774PWR, IC3 SN74AVC4T774PWR, IC4 SN74AVC4T774PWR, IC7 LM1117MP-1.8_NOPB, IC8 LM1117MP-1.8_NOPB, IC9 LM1117MP-1.8_NOPB, J4 2985-6004, J5 2985-6004, Q10 BSH103,235, Q11 BSH103,235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

Commit message: Add files via upload
Parts:
- added R1, R3, R5: 15k, SparkFun-Resistors:15KOHM-0603-1/10W-1%
- added R2, R4, R6: 6.8k, SparkFun-Resistors:6.8KOHM-0603-1/10W-1%
- C14, C16, C18: value 10uF -> 100uF
- IC7, IC8, IC9: value LM1117MP-1.8_NOPB -> LM1117IMPX-ADJ/NOPB
- renumbered JP11 to FLASH, JP12 to USB-UART, JP9 to SD_CARD
Connections:
- net GND: now also R1.1, R2.1, R2.2, R3.1, R4.1, R4.2, R5.1, R6.1, R6.2
- net VDD_1.8_1: now also R1.2
- net VDD_1.8_2: now also R3.2
- net VDD_1.8_3: now also R5.2
Other:
- moved on the sheet: C13, C15, C17, D4, IC7, R46
