File: SERV_Open8_ROHM_PCB/serv_open8_rohm.brd (EAGLE design)
At the start: 179.5 x 162.5 mm, 185 parts, among them IC1 SN74LVC1GU04DBVR, IC10 TXB0108PWR, IC11 TXB0108PWR, IC2 SN74LVC1GU04DBVR, IC3 TXB0108PWR, IC4 TXB0108PWR, IC5 TXB0108PWR, IC6 TXB0108PWR, IC7 TXB0108PWR, IC8 TXB0108PWR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

Commit message: Change in position of Jtag connector
Parts:
- moved FLASH_SERV 2.50 mm to (-82.5, -12.5)
- moved USB-UART_SERV_1 2.00 mm to (-81.0, 34.0)
- moved USB-UART_SERV_2 2.00 mm to (-81.0, 41.6)
Routing:
- net GND: track 1789.6 -> 1751.3 mm
- net VDD_3V3: track 1049.1 -> 1052.3 mm
- net VDD_5V: track 398.9 -> 400.9 mm
- net SERV_FLASH_COPI: track 21.4 -> 23.0 mm
- net SERV_UART_RX: track 13.2 -> 14.7 mm
- net SERV_FLASH_SCK: track 16.2 -> 17.3 mm
- net SERV_FLASH_CS: track 18.8 -> 19.9 mm
- net SERV_FLASH_CIPO: track 16.5 -> 17.5 mm
- net SERV_UART_TX: track 8.34 -> 7.51 mm
