File: SERV_Open8_ROHM_PCB/serv_open8_rohm.sch (EAGLE design)
At the start: 185 parts, among them IC1 SN74LVC1GU04DBVR, IC10 TXB0108PWR, IC11 TXB0108PWR, IC2 SN74LVC1GU04DBVR, IC3 TXB0108PWR, IC4 TXB0108PWR, IC5 TXB0108PWR, IC6 TXB0108PWR, IC7 TXB0108PWR, IC8 TXB0108PWR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

Commit message: Change in position of Jtag connector
Other:
- note removed: "Regulator - 5V to 1.2V"
Changed lines of the file:
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@@
 <sheet>
 <plain>
-<text x="-242.92" y="-94.43" size="1.778" layer="91">Regulator - 5V to 1.2V</text>
 <text x="-248.92" y="-38.1" size="2.54" layer="91">POWER</text>
-<text x="-230.22" y="-508.45" size="1.778" layer="91">Regulator - 5V to 1.2V</text>
 <text x="177.8" y="-434.34" size="2.54" layer="91">CLOCK GENERATOR</text>
 <text x="53.34" y="193.04" size="2.54" layer="91">RESET</text>
