File: SERV_Open8_TSMC_PCB/serv_open8_tsmc.brd (EAGLE design)
At the start: 160.5 x 179 mm, 205 parts, among them IC1 SN74LVC1GU04DBVR, IC2 SN74LVC1GU04DBVR, J4 2985-6004, Q1 BSH103,235, Q10 BSH103,235, Q11 BSH103,235, Q14 BSH103,235, Q15 BSH103,235, Q16 BSH103,235, Q17 BSH103,235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

Commit message: Change in position of Jtag connector
Parts:
- moved JTAG_OPEN8 4.00 mm to (71.0, 43.7)
Routing:
- net GND: track 1939.1 -> 1976.0 mm
- net VDD_3V3: track 1316.8 -> 1314.0 mm
- net I_TMS: track 56.3 -> 58.0 mm
- net I_TDI: track 61.7 -> 63.4 mm
- net I_TCK: track 52.4 -> 54.1 mm
