File: PCB_ROHM_BaAnh/PCB_ROHM_BaAnh.sch (EAGLE design)
At the start: 185 parts, among them IC1 TXB0108PWR, IC2 TXB0108PWR, IC3 TPS76201DBVR, IC4 TXB0108PWR, IC5 TPS76201DBVR, IC6 TXB0108PWR, IC7 TPS76201DBVR, Q1 BSH103,235, Q10 BSH103,235, Q11 BSH103,235, Q12 BSH103,235, Q13 BSH103,235, Q14 BSH103,235, Q15 BSH103,235, Q16 BSH103,235, Q17 BSH103,235, Q18 BSH103,235, Q19 BSH103,235, Q2 BSH103,235, Q20 BSH103,235, Q21 BSH103,235, Q3 BSH103,235, Q4 BSH103,235, Q5 BSH103,235, Q6 BSH103,235, Q7 BSH103,235, Q8 BSH103,235, Q9 BSH103,235

Commit message: Update PCB of Dao, change switch resistor to 0805
Parts:
- removed S1_DIP1, S1_DIP2: 219-8LPST, SamacSys_Parts:219-8LPST
- removed SWITCH: (no value), pinhead:PINHD-2X16
- added H5, H6: MOUNT-HOLE3.3, holes:MOUNT-HOLE3.3
- added JP1: (no value), pinhead:PINHD-2X16
- added S1, S2: 219-8LPST, SamacSys_Parts:219-8LPST
- R25, R26, R27, R28, R29, R30, R31, R32, R33, R34, R35, R36, R53, R54, R55, R56: device SparkFun-Resistors:10KOHM-0603-1/10W-1% -> SparkFun-Resistors:0.3OHM-0805-1/8W-1%
- renumbered CLOCKCTRL_0_CLK0 to CLOCKCTRL_0, CLOCKCTRL_1_CLK0 to CLOCKCTRL_1, CLOCKCTRL_2_CLK0 to CLOCKCTRL_2
Connections:
- net GND: now also S1.10, S1.11, S1.12, S1.13, S1.14, S1.15, S1.16, S1.9, S2.10, S2.11, S2.12, S2.13, S2.14, S2.15, S2.16, S2.9; no longer S1_DIP1.10, S1_DIP1.11, S1_DIP1.12, S1_DIP1.13, S1_DIP1.14, S1_DIP1.15, S1_DIP1.16, S1_DIP1.9, S1_DIP2.10, S1_DIP2.11, S1_DIP2.12, S1_DIP2.13, S1_DIP2.14, S1_DIP2.15, S1_DIP2.16, S1_DIP2.9
- net GPIO_IN[0]: now also JP1.31; no longer SWITCH.31
- net GPIO_IN[10]: now also JP1.11; no longer SWITCH.11
- net GPIO_IN[11]: now also JP1.9; no longer SWITCH.9
- net GPIO_IN[12]: now also JP1.7; no longer SWITCH.7
- net GPIO_IN[13]: now also JP1.5; no longer SWITCH.5
- net GPIO_IN[14]: now also JP1.3; no longer SWITCH.3
- net GPIO_IN[15]: now also JP1.1; no longer SWITCH.1
- net GPIO_IN[1]: now also JP1.29; no longer SWITCH.29
- net GPIO_IN[2]: now also JP1.27; no longer SWITCH.27
- net GPIO_IN[3]: now also JP1.25; no longer SWITCH.25
- net GPIO_IN[4]: now also JP1.23; no longer SWITCH.23
- net GPIO_IN[5]: now also JP1.21; no longer SWITCH.21
- net GPIO_IN[6]: now also JP1.19; no longer SWITCH.19
- net GPIO_IN[7]: now also JP1.17; no longer SWITCH.17
- net GPIO_IN[8]: now also JP1.15; no longer SWITCH.15
- net GPIO_IN[9]: now also JP1.13; no longer SWITCH.13
- net N$48: now also JP1.32, R33.2, S2.8; no longer R31.1, S1_DIP1.2, SWITCH.4
- net N$49: now also JP1.30, R34.2, S2.7; no longer R30.1, S1_DIP1.3, SWITCH.6
- net N$50: now also JP1.28, R35.2, S2.6; no longer R29.1, S1_DIP1.4, SWITCH.8
- net N$51: now also JP1.26, R36.2, S2.5; no longer R28.1, S1_DIP1.5, SWITCH.10
- net N$56: now also JP1.24, R53.2, S2.4; no longer R27.1, S1_DIP1.6, SWITCH.12
- net N$57: now also JP1.22, R54.2, S2.3; no longer R26.1, S1_DIP1.7, SWITCH.14
- net N$58: now also JP1.20, R55.2, S2.2; no longer R25.1, S1_DIP1.8, SWITCH.16
- net N$60: now also JP1.18, R56.2, S2.1; no longer R32.1, S1_DIP1.1, SWITCH.2
- net N$66: now also JP1.16, R25.2, S1.8; no longer R55.1, S1_DIP2.2, SWITCH.20
- net N$67: now also JP1.14, R26.2, S1.7; no longer R54.1, S1_DIP2.3, SWITCH.22
- net N$68: now also JP1.12, R27.2, S1.6; no longer R53.1, S1_DIP2.4, SWITCH.24
- net N$69: now also JP1.10, R28.2, S1.5; no longer R36.1, S1_DIP2.5, SWITCH.26
- net N$72: now also JP1.8, R29.2, S1.4; no longer R35.1, S1_DIP2.6, SWITCH.28
- net N$73: now also JP1.6, R30.2, S1.3; no longer R34.1, S1_DIP2.7, SWITCH.30
- net N$74: now also JP1.4, R31.2, S1.2; no longer R33.1, S1_DIP2.8, SWITCH.32
- net N$75: now also JP1.2, R32.2, S1.1; no longer R56.1, S1_DIP2.1, SWITCH.18
- net VDD_3V3: now also R25.1, R26.1, R27.1, R28.1, R29.1, R30.1, R31.1, R32.1, R33.1, R34.1, R35.1, R36.1, R53.1, R54.1, R55.1, R56.1; no longer R25.2, R26.2, R27.2, R28.2, R29.2, R30.2, R31.2, R32.2, R33.2, R34.2, R35.2, R36.2, R53.2, R54.2, R55.2, R56.2
Other:
- moved on the sheet: R25, R26, R27, R28, R29, R30, R31, R32, R33, R34, R35, R36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
