File: PCB_Rocket32_TRASIO/Rocket32_TRASIO.brd (EAGLE design)
At the start: 154.9 x 111.8 mm, 67 parts, among them IC1 TXB0108PWR, IC2 TXB0108PWR, IC3 AMS1117-1.8, IC5 AMS1117-1.8, J1 2985-6004, J2 2985-6004, J4 2985-6004, J5 2985-6004, Q1 BSH103,235, Q2 BSH103,235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

Commit message: Update the new n channel mosfet
Parts:
- removed Q1, Q2, Q3, Q4: BSH103,235, SamacSys_Parts:SOT95P230X110-3N
- added Q5, Q6, Q7, Q8: 2N7002K-7, SamacSys_Parts:SOT96P240X100-3N
Connections:
- removed net N$43: D1.C, Q4.3
- removed net N$55: D2.C, Q1.3
- removed net N$57: D3.C, Q2.3
- removed net N$59: D4.C, Q3.3
- new net N$17: D4.C, Q5.3
- new net N$18: D2.C, Q6.3
- new net N$19: D3.C, Q7.3
- new net N$20: D1.C, Q8.3
- net GND: now also Q5.2, Q6.2, Q7.2, Q8.2; no longer Q1.2, Q2.2, Q3.2, Q4.2
- net GPIO_OUT[0]: now also Q7.1; no longer Q2.1
- net VDDO_LED: now also Q6.1; no longer Q1.1
- net VDD_3V3: now also Q5.1; no longer Q3.1
- net VDD_LED: now also Q8.1; no longer Q4.1
Routing:
- net GND: track 918.5 -> 910.7 mm
- net N$20: track 0.00 -> 2.86 mm
- net N$19: track 0.00 -> 2.86 mm
- net N$17: track 0.00 -> 2.86 mm
- net N$18: track 0.00 -> 2.86 mm
- net N$59: track 2.81 -> 0.00 mm
- net N$43: track 2.81 -> 0.00 mm
- net N$57: track 2.81 -> 0.00 mm
- net N$55: track 2.81 -> 0.00 mm
