File: PCB_Rocket32_TRASIO/Rocket32_TRASIO.sch (EAGLE design)
At the start: 67 parts, among them IC1 TXB0108PWR, IC2 TXB0108PWR, IC3 AMS1117-1.8, IC5 AMS1117-1.8, J1 2985-6004, J2 2985-6004, J4 2985-6004, J5 2985-6004, Q1 BSH103,235, Q2 BSH103,235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

Commit message: Update the new n channel mosfet
Parts:
- removed Q1, Q2, Q3, Q4: BSH103,235, SamacSys_Parts:BSH103,235
- added Q5, Q6, Q7, Q8: 2N7002K-7, SamacSys_Parts:2N7002K-7
Connections:
- removed net N$43: D1.C, Q4.D
- removed net N$55: D2.C, Q1.D
- removed net N$57: D3.C, Q2.D
- removed net N$59: D4.C, Q3.D
- new net N$17: D4.C, Q5.D
- new net N$18: D2.C, Q6.D
- new net N$19: D3.C, Q7.D
- new net N$20: D1.C, Q8.D
- net GND: now also Q5.S, Q6.S, Q7.S, Q8.S; no longer Q1.S, Q2.S, Q3.S, Q4.S
- net GPIO_OUT[0]: now also Q7.G; no longer Q2.G
- net VDDO_LED: now also Q6.G; no longer Q1.G
- net VDD_3V3: now also Q5.G; no longer Q3.G
- net VDD_LED: now also Q8.G; no longer Q4.G
Other:
- moved on the sheet: D1, D2, D3, D4, R10, R11, R12, R13, R14, R15, R16, R17
