File: PCB_SOTB_Feb2022/SOTB_Feb22.sch (EAGLE design)
At the start: 110 parts, among them IC1 LP38511MR-ADJ_NOPB, IC2 LP38511MR-ADJ_NOPB, IC3 LP38511MR-ADJ_NOPB, IC4 SN74LVC1GU04DCKR, IC5 SN74LVC1G14DCKR, J1 2985-6004, J2 2985-6004, Y1 NX3225GA-12MHZ-STD-CRG-2

Commit message: Update the PCB with layout
Parts:
- removed H4: MOUNT-HOLE3.3, holes:MOUNT-HOLE3.3
- removed LED8: (no value), led:LEDCHIPLED_1206
- removed R19: 1k, Resistor:R_CHIP-1206(3216-METRIC)
- removed USB-UART_1: PINHD-1X4, Connector:PINHD-1X4
- added C40: 2.7pF, Capacitor:C_CHIP-1206(3216-METRIC)
- added L1: LQG15HS1N8S02D, SamacSys_Parts:LQG15HS1N8S02D
- added SERV_UART: PINHD-1X4, Connector:PINHD-1X4
- added SJ1: (no value), jumper:SJ
- added U$1: (no value), DN024_TI_ANTENNA:868MHZA_ANTENNA_DN024
- renumbered K_LOADED_RST to K_LD_RST, LED1 to DY_LEDS, LED2 to K_OLEDG[0], SERV_RST1 to RS_RST, USB-UART_3 to RS_UART
Connections:
- removed net IN_0.8: C1.1, IC1.EN, IC1.IN_1, IC1.IN_2
- removed net IN_1.2: C4.1, IC2.EN, IC2.IN_1, IC2.IN_2
- removed net VSSQ: SOCKET.67
- new net N$27: L1.2, U$1.P$1
- new net N$28: SERV_LORA.ANT, SJ1.1
- net DY_ALL_RX_IN: now also SERV_UART.2; no longer USB-UART_1.2
- net DY_ALL_TX_OUT: now also SERV_UART.4; no longer USB-UART_1.4
- net GND: now also C40.2, SERV_UART.1, SOCKET.67; no longer R19.1, USB-UART_1.1
- net IN_3.3: now also C1.1, C4.1, IC1.EN, IC1.IN_1, IC1.IN_2, IC2.EN, IC2.IN_1, IC2.IN_2
- net N$26: now also C40.1, L1.1, SJ1.2; no longer LED8.C, R19.2
- net VDD_3.3V: now also SERV_UART.3; no longer USB-UART_1.3
- net VDD_5V_UART: no longer LED8.A
Other:
- note added: "SOTB Feb. 2022 Copyright © UEC PHAM LAB 2022 SERV RV32E LEROS OLINGUITO + TRNG"
- note removed: "SOTB Feb. 2022 Copyright © UEC PHAM LAB 2022 SERV 32RVE LEROS OLINGUITO + TRNG"
- moved on the sheet: SERV_LORA, USB-UART_2
