File: PCB_ROHM_102022/ROHM_102022.sch (EAGLE design)
At the start: 126 parts, among them IC1 AMS1117-1.8, IC10 TXB0108PWR, IC2 TXB0108PWR, IC3 W9825G6KH-6I, IC4 AMS1117-1.8, IC5 AMS1117-1.8, IC7 TXB0108PWR, J1 2985-6004, J2 2985-6004, J3 2985-6004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

Commit message: Update pdf for schematic of ROHM102022
Other:
- note added: "DLDO & PUF"
- note added: "LEROS"
- note added: "MEMORY"
- note added: "POWER"
- note added: "ROCKET"
- note added: "ROCKET_FPGA"
- note added: "SERV"
- note added: "SOCKET"
- note removed: "JTAG"
Changed lines of the file:
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@@
 <sheet>
 <plain>
-<text x="-308.356" y="-147.828" size="6.4516" layer="91">JTAG</text>
 <text x="-298.54" y="-464.02" size="2.54" layer="91">SERV_JTAG</text>
 <text x="-328.7" y="-587.03" size="2.54" layer="91">SERV_FLASH</text>
 <text x="-7.834" y="-604.844" size="2.54" layer="91">SMA</text>
 <text x="311.444" y="-366.084" size="2.54" layer="91">SMA</text>
+<text x="-343.94" y="-330.49" size="6.4516" layer="91">SERV</text>
+<text x="171.68" y="-340.65" size="6.4516" layer="91">LEROS</text>
+<text x="-335.28" y="119.38" size="6.4516" layer="91">SOCKET</text>
+<text x="101.6" y="116.84" size="6.4516" layer="91">MEMORY</text>
+<text x="335.28" y="116.84" size="6.4516" layer="91">DLDO &amp; PUF</text>
+<text x="487.68" y="116.84" size="6.4516" layer="91">ROCKET_FPGA</text>
+<text x="347.98" y="-144.78" size="6.4516" layer="91">POWER</text>
+<text x="-281.94" y="-139.7" size="6.4516" layer="91">ROCKET</text>
 </plain>
 <instances>

Commit message: Connect JTAG to FPGA
Parts:
- removed C1, C2: 0.1uF, SparkFun-Capacitors:10UF-1206-6.3V-20%
- removed IC2: TXB0108PWR, SamacSys_Parts:TXB0108PWR
- removed JTAG_20_PIN: (no value), pinhead:PINHD-2X10
- removed ROCKET_JTAG: PINHD-2X5, Connector:PINHD-2X5
- added JTAG_TCK: (no value), pinhead:PINHD-1X2
- ROCKET_FPGA: device pinhead:PINHD-2X15 -> pinhead:PINHD-2X17
Connections:
- removed net N$2: IC2.A8, ROCKET_JTAG.10
- removed net N$6: IC2.A7, ROCKET_JTAG.8
- removed net N$7: IC2.A6, ROCKET_JTAG.6
- removed net N$8: IC2.A5, ROCKET_JTAG.4
- removed net N$9: IC2.A4, ROCKET_JTAG.2
- removed net TDI: IC2.B6, JTAG_20_PIN.5
- removed net TDO: IC2.B4, JTAG_20_PIN.13
- removed net TMS: IC2.B8, JTAG_20_PIN.7
- removed net TRSTN: IC2.B5, JTAG_20_PIN.3
- net GND: no longer C1.2, C2.2, JTAG_20_PIN.10, JTAG_20_PIN.12, JTAG_20_PIN.14, JTAG_20_PIN.16, JTAG_20_PIN.18, JTAG_20_PIN.20, JTAG_20_PIN.4, JTAG_20_PIN.6, JTAG_20_PIN.8
- net JTAG_TCK: now also JTAG_TCK.1; no longer ROCKET_JTAG.7
- net JTAG_TDI: now also ROCKET_FPGA.32; no longer ROCKET_JTAG.5
- net JTAG_TDO: now also ROCKET_FPGA.34; no longer ROCKET_JTAG.1
- net JTAG_TMS: now also ROCKET_FPGA.28; no longer ROCKET_JTAG.9
- net JTAG_TRSTN: now also ROCKET_FPGA.33; no longer ROCKET_JTAG.3
- net TCK: now also JTAG_TCK.2, ROCKET_FPGA.31; no longer IC2.B7, JTAG_20_PIN.9
- net VDD_1.8_IO: no longer C1.1, IC2.OE, IC2.VCCA
- net VDD_3V3: no longer C2.1, IC2.GND, IC2.VCCB, JTAG_20_PIN.1, JTAG_20_PIN.2

Commit message: Upload bom and cpl
Parts:
- removed D1, D2, D3, D4: LED0, SparkFun-LED:LED0603
- removed JTAG_TCK: (no value), pinhead:PINHD-1X2
- removed Q1, Q2, Q3, Q4: BSH103,235, SamacSys_Parts:BSH103,235
- removed R10, R12, R13, R15, R16, R17, R8: 10k, SparkFun-Resistors:10OHM-1206-1/4W-1%
- removed R7, R9: 330, SparkFun-Resistors:10OHM-1206-1/4W-1%
- added J5: (no value), SparkFun-Connectors:CONN_03
- added J6: (no value), SparkFun-Connectors:CONN_05X2PTH
- added JP1: (no value), pinhead:PINHD-1X3
- added JTAG_ROCKET: (no value), pinhead:PINHD-2X10
- added LED1, LED2, LED3, LED4, LOADED: (no value), adafruit:LEDCHIPLED_0805
- added R11: 10k, SparkFun-Resistors:10OHM-1206-1/4W-1%
- added S3: SS12SDP2, SamacSys_Parts:SS12SDP2
- R14, R4, R6: value 10k -> 330; device SparkFun-Resistors:10OHM-1206-1/4W-1% -> Resistor:R_CHIP-1206(3216-METRIC)
- R3, R5: device SparkFun-Resistors:10OHM-1206-1/4W-1% -> Resistor:R_CHIP-1206(3216-METRIC)
Connections:
- removed net N$16: D1.A, R5.1
- removed net N$17: D1.C, Q1.D
- removed net N$18: D2.A, R7.1
- removed net N$19: D2.C, Q2.D
- removed net N$20: D4.A, R9.1
- removed net N$21: D4.C, Q3.D
- removed net TCK: JTAG_TCK.2, ROCKET_FPGA.31
- new net JTAG_TCK_FPGA: J6.3, ROCKET_FPGA.31
- new net JTAG_TDI_FPGA: J6.5, ROCKET_FPGA.32
- new net JTAG_TDO_FPGA: J6.9, ROCKET_FPGA.34
- new net JTAG_TMS_FPGA: J6.1, ROCKET_FPGA.28
- new net JTAG_TRSTN_FPGA: J6.7, ROCKET_FPGA.33
- new net LEROS_PAD_LOADER_RST_N_0_FPGA: FPGA_LEROS.4, JP1.1
- new net LEROS_PAD_SRAM_LOADED_0_FPGA: FPGA_LEROS.12, J5.1
- new net N$2: LED1.C, R14.2
- new net N$6: JP1.3, R11.1, S3.COM
- new net N$7: LED2.C, R3.2
- new net N$8: LED3.C, R4.2
- new net N$9: LED4.C, R5.2
- net GND: now also JTAG_ROCKET.10, JTAG_ROCKET.12, JTAG_ROCKET.14, JTAG_ROCKET.16, JTAG_ROCKET.18, JTAG_ROCKET.20, JTAG_ROCKET.4, JTAG_ROCKET.6, JTAG_ROCKET.8, R3.1, R5.1, S3.ON_2; no longer Q1.S, Q2.S, Q3.S, Q4.S, R10.1, R12.1, R13.1, R15.1, R16.1, R17.1, R8.1
- net JTAG_TCK: now also J6.4, JTAG_ROCKET.9; no longer JTAG_TCK.1
- net JTAG_TDI: now also J6.6, JTAG_ROCKET.5; no longer ROCKET_FPGA.32
- net JTAG_TDO: now also J6.10, JTAG_ROCKET.13; no longer ROCKET_FPGA.34
- net JTAG_TMS: now also J6.2, JTAG_ROCKET.7; no longer ROCKET_FPGA.28
- net JTAG_TRSTN: now also J6.8, JTAG_ROCKET.3; no longer ROCKET_FPGA.33
- net LEROS_PAD_LOADER_RST_N_0: now also JP1.2; no longer FPGA_LEROS.4
- net LEROS_PAD_OLEDG_0_0: now also LED1.A; no longer Q4.G, R4.2
- net LEROS_PAD_OLEDG_0_1: now also LED2.A; no longer Q1.G, R6.2
- net LEROS_PAD_OLEDG_0_2: now also LED3.A; no longer Q2.G, R8.2
- net LEROS_PAD_OLEDG_0_3: now also LED4.A; no longer Q3.G, R10.2
- net LEROS_PAD_SRAM_LOADED_0: now also J5.2; no longer FPGA_LEROS.12
- net N$14: now also LOADED.C, R6.2; no longer D3.C, Q4.D
- net N$15: now also J5.3, LOADED.A; no longer D3.A, R3.1
- net SERV_MOD_IO_ALL_DIPSW_PAD_ALL_DIPSW_0_0: no longer R17.2
- net SERV_PAD_ALL_LEDS_0_0: no longer R15.2
- net SERV_PAD_ALL_LEDS_0_1: no longer R16.2
- net SERV_SPI_COPI: no longer R12.2
- net SERV_SPI_CS: no longer R14.2
- net SERV_SPI_SCK: no longer R13.2
- net VDD_3V3: now also JTAG_ROCKET.1, JTAG_ROCKET.2, R11.2, S3.ON_1; no longer R3.2, R5.2, R7.2, R9.2
Other:
- note added: "3 regulators of 1.8V Supply of 3.3V is from UART for SERV or GPIO for LEROS and Rocket"
- note added: "32kHz"
- note added: "50MHz"
- note added: "Only 4 Leds is implemented to save space"
- note added: "ROCKET_JTAG"
- note added: "ROHM 2022 ROCKET_SERV LEROS DLDO_PUF Copyright © UEC Pham Lab"
- note added: "This connector is connected to the last 12 pin of 40 pin GPIO connector"
- note added: "W9825G6KH-6I SDRAM from Winbond 32MB"
- moved on the sheet: 3.3V_MUX, C10, C11, C12, C13, C14, C15, C16, C17, C18, C19, C20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
