File: PCB_SOTB_LWC/SOTB_LWC.sch (EAGLE design)
At the start: 99 parts, among them IC1 LP38511MR-ADJ_NOPB, IC2 LP38511MR-ADJ_NOPB, IC3 LP38511MR-ADJ_NOPB, IC4 SN74LVC1GU04DCKR, IC5 SN74LVC1G14DCKR, J1 2985-6004, Y2 Q13FC1350000400

Commit message: Change led from 1206 to 0805
Parts:
- LED3, LED4, LED5, LW_O0, LW_O1: device led:LEDCHIPLED_1206 -> led:LEDCHIPLED_0805
